File: hardware/sensor.sch (EAGLE design)
At the start: 11 parts, among them Q1 2N7000KL/BS170KL

Commit message: board changes
Parts:
- removed Q1: 2N7000KL/BS170KL, m-pad-2.1:2N7000KL/BS170KL
- removed U$2: BATTERY-CHARGER-LI-5V, diy-modules:BATTERY-CHARGER-LI-5V
- added PWRC: 2N7000, 2N7000:2N7000
Connections:
- new net N$3: PWRC.S
- new net N$4: PWRC.D
- net EXT_GND: no longer Q1.S
- net GND: no longer Q1.D
- net SENS_EN: now also PWRC.G; no longer Q1.G
Other:
- moved on the sheet: JP3
Changed lines of the file:
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@@
 <part name="SW_RST" library="con-amp-quick" library_urn="urn:adsk.eagle:library:125" deviceset="M02" device="" package3d_urn="urn:adsk.eagle:package:5956/1" value="2"/>
 <part name="SUPPLY1" library="SparkFun-PowerSymbols" library_urn="urn:adsk.eagle:library:530" deviceset="3.3V" device=""/>
-<part name="U$2" library="diy-modules" deviceset="BATTERY-CHARGER-LI-5V" device=""/>
 <part name="DS18B1" library="con-amp-quick" library_urn="urn:adsk.eagle:library:125" deviceset="M03" device="" package3d_urn="urn:adsk.eagle:package:5957/1"/>
 <part name="DS18B2" library="con-amp-quick" library_urn="urn:adsk.eagle:library:125" deviceset="M03" device="" package3d_urn="urn:adsk.eagle:package:5957/1"/>
-<part name="Q1" library="m-pad-2.1" deviceset="2N7000KL/BS170KL" device=""/>
 <part name="V1" library="m-pad-2.1" deviceset="GND" device=""/>
+<part name="PWRC" library="2N7000" deviceset="2N7000" device=""/>
+<part name="EXTGND" library="m-pad-2.1" deviceset="GND" device=""/>
 </parts>
 <sheets>
@@
 <attribute name="VALUE" x="-82.55" y="619.76" size="1.778" layer="96"/>
 </instance>
-<instance part="JP3" gate="A" x="43.18" y="637.54" smashed="yes">
-<attribute name="NAME" x="41.91" y="658.495" size="1.778" layer="95"/>
-<attribute name="VALUE" x="36.83" y="617.22" size="1.778" layer="96"/>
+<instance part="JP3" gate="A" x="15.24" y="637.54" smashed="yes">
+<attribute name="NAME" x="13.97" y="658.495" size="1.778" layer="95"/>
+<attribute name="VALUE" x="8.89" y="617.22" size="1.778" layer="96"/>
 </instance>
 <instance part="DHT22" gate="A" x="-15.24" y="655.32" smashed="yes" rot="R90">
@@
 <attribute name="NAME" x="-41.402" y="640.08" size="1.778" layer="95" rot="R90"/>
 </instance>
-<instance part="SUPPLY1" gate="G$1" x="-88.9" y="576.58" smashed="yes">
-<attribute name="VALUE" x="-88.9" y="579.374" size="1.778" layer="96" align="bottom-center"/>
-</instance>
-<instance part="U$2" gate="G$1" x="-68.58" y="566.42" smashed="yes">
-<attribute name="NAME" x="-78.74" y="581.66" size="1.778" layer="95"/>
-<attribute name="VALUE" x="-78.74" y="579.12" size="1.778" layer="96"/>
+<instance part="SUPPLY1" gate="G$1" x="-20.32" y="584.2" smashed="yes">
+<attribute name="VALUE" x="-20.32" y="586.994" size="1.778" layer="96" align="bottom-center"/>
 </instance>
 <instance part="DS18B1" gate="G$1" x="-2.54" y="599.44" smashed="yes" rot="R90">
@@
 <attribute name="NAME" x="-23.622" y="596.9" size="1.778" layer="95" rot="R90"/>
 </instance>
-<instance part="Q1" gate="G$1" x="20.32" y="607.06" smashed="yes">
-<attribute name="VALUE" x="26.67" y="608.33" size="1.778" layer="96"/>
-<attribute name="NAME" x="26.67" y="610.87" size="1.778" layer="95"/>
-</instance>
-<instance part="V1" gate="GND" x="38.1" y="591.82" smashed="yes">
-<attribute name="VALUE" x="36.195" y="588.01" size="1.778" layer="96"/>
+<instance part="V1" gate="GND" x="10.16" y="589.28" smashed="yes">
+<attribute name="VALUE" x="8.255" y="585.47" size="1.778" layer="96"/>
+</instance>
+<instance part="PWRC" gate="G$1" x="55.88" y="645.16" smashed="yes">
+<attribute name="NAME" x="60.96" y="645.16" size="1.778" layer="95"/>
+<attribute name="VALUE" x="60.96" y="641.35" size="1.778" layer="96"/>
+</instance>
+<instance part="EXTGND" gate="GND" x="27.94" y="589.28" smashed="yes">
+<attribute name="VALUE" x="26.035" y="585.47" size="1.778" layer="96"/>
 </instance>
 </instances>
@@
 <segment>
 <pinref part="JP3" gate="A" pin="11"/>
-<wire x1="40.64" y1="627.38" x2="25.4" y2="627.38" width="0.1524" layer="91"/>
-<label x="26.416" y="627.888" size="1.778" layer="95"/>
-<junction x="40.64" y="627.38"/>
+<wire x1="12.7" y1="627.38" x2="25.4" y2="627.38" width="0.1524" layer="91"/>
+<label x="18.034" y="627.634" size="1.778" layer="95"/>
+<junction x="12.7" y="627.38"/>
 </segment>
 </net>
@@
 <pinref part="DHT22" gate="A" pin="2"/>
 <wire x1="-15.24" y1="652.78" x2="-15.24" y2="632.46" width="0.1524" layer="91"/>
-<wire x1="-15.24" y1="632.46" x2="40.64" y2="632.46" width="0.1524" layer="91"/>
+<wire x1="-15.24" y1="632.46" x2="12.7" y2="632.46" width="0.1524" layer="91"/>
 <junction x="-15.24" y="652.78"/>
 <label x="-14.478" y="657.86" size="1.778" layer="95" rot="R90"/>
-<label x="25.4" y="632.968" size="1.778" layer="95"/>
-<junction x="40.64" y="632.46"/>
+<label x="18.034" y="631.698" size="1.778" layer="95"/>
+<junction x="12.7" y="632.46"/>
 </segment>
 </net>
@@
 <junction x="-48.26" y="607.06"/>
 <label x="-45.72" y="612.14" size="1.778" layer="95" rot="R90"/>
-</segment>
-<segment>
-<pinref part="Q1" gate="G$1" pin="D"/>
-<junction x="22.86" y="612.14"/>
-<label x="25.4" y="617.22" size="1.778" layer="95" rot="R180"/>
 </segment>
 <segment>
@@
 <net name="EXT_GND" class="0">
 <segment>
-<pinref part="Q1" gate="G$1" pin="S"/>
-<junction x="22.86" y="601.98"/>
-<label x="22.86" y="594.36" size="1.778" layer="95" rot="R90"/>
-</segment>
-<segment>
 <pinref part="JP3" gate="A" pin="8"/>
-<wire x1="40.64" y1="635" x2="-5.08" y2="635" width="0.1524" layer="91"/>
-<label x="23.368" y="636.016" size="1.778" layer="95"/>
-<junction x="40.64" y="635"/>
+<wire x1="12.7" y1="635" x2="-5.08" y2="635" width="0.1524" layer="91"/>
+<label x="18.034" y="634.492" size="1.778" layer="95"/>
+<junction x="12.7" y="635"/>
+</segment>
+</net>
+<net name="N$3" class="0">
+<segment>
+<pinref part="PWRC" gate="G$1" pin="S"/>
+<junction x="58.42" y="637.54"/>
+</segment>
+</net>
+<net name="N$4" class="0">
+<segment>
+<pinref part="PWRC" gate="G$1" pin="D"/>
+<junction x="58.42" y="650.24"/>
 </segment>
 </net>
@@
 <segment>
 <pinref part="JP3" gate="A" pin="5"/>
-<wire x1="40.64" y1="642.62" x2="25.4" y2="642.62" width="0.1524" layer="91"/>
-<junction x="40.64" y="642.62"/>
-<label x="22.606" y="643.636" size="1.778" layer="95"/>
-</segment>
-<segment>
-<pinref part="Q1" gate="G$1" pin="G"/>
-<junction x="15.24" y="604.52"/>
-<label x="5.08" y="607.06" size="1.778" layer="95"/>
-<wire x1="15.24" y1="604.52" x2="10.16" y2="604.52" width="0.1524" layer="91"/>
-</segment>
-</net>
+<wire x1="50.8" y1="642.62" x2="12.7" y2="642.62" width="0.1524" layer="91"/>
+<junction x="12.7" y="642.62"/>
+<label x="45.72" y="640.08" size="1.778" layer="95"/>
+<pinref part="PWRC" gate="G$1" pin="G"/>
+</segment>
+</net>

Commit message: board changes
Parts:
- renumbered DS18B20 to DS18B0
Connections:
- net N$4 renamed EXTGND
- removed net N$3: PWRC.S
- net 1WIRE: now also DS18B0.3; no longer DS18B0.2
- net 3.3V: now also DS18B0.1; no longer DS18B0.3
- net GND: now also DS18B0.2, PWRC.S; no longer DS18B0.1
Changed lines of the file:
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@@
 <parts>
 <part name="FRAME1" library="frames" library_urn="urn:adsk.eagle:library:229" deviceset="A4-35SC" device=""/>
-<part name="DS18B20" library="con-amp-quick" library_urn="urn:adsk.eagle:library:125" deviceset="M03" device="" package3d_urn="urn:adsk.eagle:package:5957/1"/>
+<part name="DS18B0" library="con-amp-quick" library_urn="urn:adsk.eagle:library:125" deviceset="M03" device="" package3d_urn="urn:adsk.eagle:package:5957/1"/>
 <part name="R1" library="resistor-power" library_urn="urn:adsk.eagle:library:344" deviceset="R" device="AC01" package3d_urn="urn:adsk.eagle:package:25124/1" value="4.7K"/>
 <part name="JP1" library="adafruit" library_urn="urn:adsk.eagle:library:420" deviceset="PINHD-1X13" device="" package3d_urn="urn:adsk.eagle:package:6240833/1"/>
@@
 <attribute name="LAST_DATE_TIME" x="17.145" y="680.593" size="1.524" layer="94" ratio="12"/>
 </instance>
-<instance part="DS18B20" gate="G$1" x="-50.8" y="599.44" smashed="yes" rot="R90">
+<instance part="DS18B0" gate="G$1" x="-50.8" y="599.44" smashed="yes" rot="R90">
 <attribute name="VALUE" x="-43.18" y="596.9" size="1.778" layer="96" rot="R90"/>
 <attribute name="NAME" x="-56.642" y="596.9" size="1.778" layer="95" rot="R90"/>
@@
 </segment>
 <segment>
-<pinref part="DS18B20" gate="G$1" pin="3"/>
-<junction x="-53.34" y="607.06"/>
-<wire x1="-53.34" y1="607.06" x2="-53.34" y2="617.22" width="0.1524" layer="91"/>
-<label x="-50.8" y="612.14" size="1.778" layer="95" rot="R90"/>
+<pinref part="DS18B0" gate="G$1" pin="1"/>
+<junction x="-48.26" y="607.06"/>
+<wire x1="-48.26" y1="607.06" x2="-48.26" y2="617.22" width="0.1524" layer="91"/>
+<label x="-45.974" y="610.616" size="1.778" layer="95" rot="R90"/>
 </segment>
 <segment>
@@
 </segment>
 <segment>
-<pinref part="DS18B20" gate="G$1" pin="1"/>
-<wire x1="-48.26" y1="607.06" x2="-48.26" y2="617.22" width="0.1524" layer="91"/>
-<junction x="-48.26" y="607.06"/>
-<label x="-45.72" y="612.14" size="1.778" layer="95" rot="R90"/>
+<pinref part="DS18B0" gate="G$1" pin="2"/>
+<wire x1="-50.8" y1="607.06" x2="-50.8" y2="617.22" width="0.1524" layer="91"/>
+<junction x="-50.8" y="607.06"/>
+<label x="-49.022" y="610.362" size="1.778" layer="95" rot="R90"/>
 </segment>
 <segment>
@@
 <label x="-1.778" y="611.886" size="1.778" layer="95" rot="R90"/>
 </segment>
+<segment>
+<pinref part="PWRC" gate="G$1" pin="S"/>
+<junction x="58.42" y="637.54"/>
+<label x="58.42" y="629.92" size="1.778" layer="95"/>
+</segment>
 </net>
 <net name="1WIRE" class="0">
@@
 <pinref part="R1" gate="G$1" pin="2"/>
 <wire x1="-68.58" y1="629.92" x2="-60.96" y2="629.92" width="0.1524" layer="91"/>
-<wire x1="-60.96" y1="629.92" x2="-50.8" y2="629.92" width="0.1524" layer="91"/>
+<wire x1="-60.96" y1="629.92" x2="-53.34" y2="629.92" width="0.1524" layer="91"/>
 <junction x="-60.96" y="629.92"/>
-<pinref part="DS18B20" gate="G$1" pin="2"/>
-<wire x1="-50.8" y1="629.92" x2="-50.8" y2="607.06" width="0.1524" layer="91"/>
-<junction x="-50.8" y="607.06"/>
-<label x="-48.26" y="612.14" size="1.778" layer="95" rot="R90"/>
+<pinref part="DS18B0" gate="G$1" pin="3"/>
+<wire x1="-53.34" y1="629.92" x2="-53.34" y2="607.06" width="0.1524" layer="91"/>
+<junction x="-53.34" y="607.06"/>
+<label x="-51.562" y="610.362" size="1.778" layer="95" rot="R90"/>
 <junction x="-68.58" y="629.92"/>
 </segment>
@@
 </segment>
 </net>
-<net name="N$3" class="0">
-<segment>
-<pinref part="PWRC" gate="G$1" pin="S"/>
-<junction x="58.42" y="637.54"/>
-</segment>
-</net>
-<net name="N$4" class="0">
+<net name="EXTGND" class="0">
 <segment>
 <pinref part="PWRC" gate="G$1" pin="D"/>
 <junction x="58.42" y="650.24"/>
-</segment>
-</net>
+<label x="55.88" y="655.32" size="1.778" layer="95"/>
+</segment>
+</net>
