File: hardware/Eagle/Vesoil/sensor.sch (EAGLE design)
At the start: 10 parts, among them J1 RJ45

Commit message: board changes
Parts:
- removed DS18B20: DS18B20, con-amp-quick:M03
- removed J1: RJ45, SparkFun-Connectors:RJ45-8
- removed SW_MODE: SW1, con-amp-quick:M02
- removed SW_RST: SW2, con-amp-quick:M02
- added MODE, RST: JST-XH-02-PIN-LONG-PAD, Rembrandt Electronics - JST XH Connectors v1-0:JST-XH-02-PIN-LONG-PAD
- added SENSOR: JST-XH-04-PIN-LONG-PAD, Rembrandt Electronics - JST XH Connectors v1-0:JST-XH-04-PIN-LONG-PAD
- added TEMP: JST-XH-03-PIN-LONG-PAD, Rembrandt Electronics - JST XH Connectors v1-0:JST-XH-03-PIN-LONG-PAD
Connections:
- net N$7 renamed SENS_ENABLE
- net 1WIRE: now also TEMP-1.S; no longer DS18B20.1
- net 3.3V: now also SENSOR-4.S, TEMP-3.S; no longer DS18B20.3, J1.3
- net GND: now also MODE-2.S, RST-1.S; no longer SW_MODE.1, SW_RST.1
- net MODE: now also JP1.2, MODE-1.S; no longer JP1.9, SW_MODE.2
- net RST: now also RST-2.S; no longer SW_RST.2
- net SCL: now also SENSOR-2.S; no longer J1.7
- net SDA: now also SENSOR-1.S; no longer J1.8
- net SENS_GND: now also SENSOR-3.S, TEMP-2.S; no longer DS18B20.2, J1.6
