File: hardware/Eagle/Vesoil/sensor.brd (EAGLE design)
At the start: 40.6 x 51.7 mm, 10 parts, among them J1 RJ45

Commit message: board changes
Parts:
- removed DS18B20: DS18B20, con-amp-quick:03P
- removed J1: RJ45, SparkFun-Connectors:RJ45-8
- removed SW_MODE: SW1, con-amp-quick:02P
- removed SW_RST: SW2, con-amp-quick:02P
- added MODE, RST: JST-XH-02-PIN-LONG-PAD, Rembrandt Electronics - JST XH Connectors v1-0:JST-XH-02-PACKAGE-LONG-PAD
- added SENSOR: JST-XH-04-PIN-LONG-PAD, Rembrandt Electronics - JST XH Connectors v1-0:JST-XH-04-PACKAGE-LONG-PAD
- added TEMP: JST-XH-03-PIN-LONG-PAD, Rembrandt Electronics - JST XH Connectors v1-0:JST-XH-03-PACKAGE-LONG-PAD
- moved MOSFET1 4.02 mm to (24.1, 77.5)
- moved DHT22 2.54 mm to (34.3, 77.5)
- moved R1 1.80 mm to (41.9, 72.4)
Connections:
- net N$7 renamed SENS_ENABLE
- net 1WIRE: now also TEMP.1; no longer DS18B20.1
- net 3.3V: now also SENSOR.4, TEMP.3; no longer DS18B20.3, J1.3
- net GND: now also MODE.2, RST.1; no longer SW_MODE.1, SW_RST.1
- net MODE: now also JP1.2, MODE.1; no longer JP1.9, SW_MODE.2
- net RST: now also RST.2; no longer SW_RST.2
- net SCL: now also SENSOR.2; no longer J1.7
- net SDA: now also SENSOR.1; no longer J1.8
- net SENS_GND: now also SENSOR.3, TEMP.2; no longer DS18B20.2, J1.6
Routing:
- net SDA: track 35.4 -> 14.6 mm
- net SCL: track 37.5 -> 18.2 mm
- net 3.3V: track 54.7 -> 47.8 mm
- net RST: track 12.8 -> 16.2 mm
- net DATA_T: track 12.7 -> 15.2 mm
- net SENS_GND: track 48.0 -> 50.3 mm
- net SENS_ENABLE: track 19.7 -> 18.6 mm
- net GND: track 67.5 -> 66.5 mm
- net 1WIRE: track 16.1 -> 17.0 mm
- added copper zone on layer 16, net GND
Other:
- board size 40.6 x 51.7 mm -> 48.2 x 46.7 mm
- board text added: "3V3"
- board text added: "GND"
- board text added: "SCL"
- board text added: "SDA"
- board text added: "Vestrong Sensor 1.0"
- board text added: "WRE"

Commit message: board changes
Parts:
- moved R2 46.8 mm to (14.0, 25.4)
- moved DHT22 46.8 mm to (24.1, 31.8)
- moved JP1 46.8 mm to (21.6, 16.5)
- moved JP2 46.8 mm to (21.6, 41.9)
- moved MODE 46.8 mm to (8.89, 5.08)
- moved MOSFET1 46.8 mm to (14.0, 31.8)
- moved R1 46.8 mm to (31.8, 26.7)
- moved RST 46.8 mm to (21.6, 5.08)
- moved SENSOR 46.8 mm to (40.6, 30.5)
- moved TEMP 46.8 mm to (35.6, 5.08)
Routing:
- added copper zone on layer 1, net GND
Other:
- board size 48.2 x 46.7 mm -> 45.7 x 46.7 mm

Commit message: board changes
Parts:
- moved R2 5.08 mm to (8.89, 25.4)
- moved MODE 1.27 mm to (10.2, 5.08)
Routing:
- net GND: track 66.5 -> 0.30 mm
- net SENS_ENABLE: track 18.6 -> 16.6 mm
- net SCL: track 18.2 -> 18.9 mm
- net MODE: track 12.0 -> 11.4 mm
