File: TT22_V10/hardware/MoistureSensor - Version1/Eagle/Vesoil/sensor.brd (EAGLE design)
At the start: 47 x 45.4 mm, 10 parts

Commit message: reorg boards
Parts:
- moved JP1 3.81 mm to (22.9, 12.7)
- moved R1 3.81 mm to (33.0, 22.9)
- moved DHT22 3.81 mm to (25.4, 27.9)
- moved MOSFET1 3.81 mm to (15.2, 27.9)
- moved R2 3.81 mm to (10.2, 21.6)
- moved SENSOR 3.81 mm to (41.9, 26.7)
- moved JP2 3.81 mm to (22.9, 38.1)
- moved MODE 1.27 mm to (11.4, 3.81)
- moved RST 1.27 mm to (22.9, 3.81)
- moved TEMP 1.27 mm to (36.8, 3.81)
Routing:
- net 3.3V: track 47.8 -> 45.3 mm
- net SENS_GND: track 50.3 -> 47.7 mm
- net 1WIRE: track 17.0 -> 14.5 mm
- net MODE: track 11.4 -> 8.91 mm
- net RST: track 15.1 -> 13.3 mm
Other:
- board size 47 x 45.4 mm -> 46.8 x 41.1 mm
