File: TT22_V10/hardware/MoistureSensor - Version2/Sensor/sensor.sch (EAGLE design)
At the start: 10 parts

Commit message: reorg boards
Connections:
- net GND: now also RST-2.S; no longer RST-1.S
- net RST: now also RST-1.S; no longer RST-2.S
Changed lines of the file:
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@@
 </segment>
 <segment>
-<pinref part="RST" gate="-2" pin="S"/>
-<wire x1="-63.5" y1="662.94" x2="-73.66" y2="662.94" width="0.1524" layer="91"/>
-<label x="-73.66" y="662.94" size="1.778" layer="95"/>
+<pinref part="RST" gate="-1" pin="S"/>
+<wire x1="-63.5" y1="665.48" x2="-73.66" y2="665.48" width="0.1524" layer="91"/>
+<label x="-73.66" y="665.48" size="1.778" layer="95"/>
 </segment>
 </net>
@@
 </segment>
 <segment>
-<pinref part="RST" gate="-1" pin="S"/>
-<wire x1="-63.5" y1="665.48" x2="-73.66" y2="665.48" width="0.1524" layer="91"/>
-<label x="-73.66" y="665.48" size="1.778" layer="95"/>
-</segment>
-<segment>
 <pinref part="MODE" gate="-2" pin="S"/>
 <wire x1="-33.02" y1="662.94" x2="-48.26" y2="662.94" width="0.1524" layer="91"/>
 <label x="-48.26" y="662.94" size="1.778" layer="95"/>
 </segment>
+<segment>
+<pinref part="RST" gate="-2" pin="S"/>
+<wire x1="-63.5" y1="662.94" x2="-73.66" y2="662.94" width="0.1524" layer="91"/>
+<label x="-73.66" y="662.94" size="1.778" layer="95"/>
+</segment>
 </net>
