File: TT22_V10/hardware/MoistureSensor - Version2/Sensor/sensor.brd (EAGLE design)
At the start: 47 x 46.7 mm, 10 parts

Commit message: reorg boards
Parts:
- moved R1 4.02 mm to (33.0, 22.9)
- moved JP1 4.02 mm to (22.9, 12.7)
- moved DHT22 4.02 mm to (25.4, 27.9)
- moved MOSFET1 4.02 mm to (15.2, 27.9)
- moved R2 4.02 mm to (10.2, 21.6)
- moved SENSOR 4.02 mm to (41.9, 26.7)
- moved JP2 4.02 mm to (22.9, 38.1)
- moved MODE 1.80 mm to (11.4, 3.81)
- moved RST 1.80 mm to (22.9, 3.81)
- moved TEMP 1.80 mm to (36.8, 3.81)
Routing:
- net SENS_GND: track 50.3 -> 47.7 mm
- net 1WIRE: track 17.0 -> 14.5 mm
- net 3.3V: track 47.8 -> 45.3 mm
- net MODE: track 11.4 -> 8.91 mm
- net RST: track 15.1 -> 13.3 mm
Other:
- board size 47 x 46.7 mm -> 46.8 x 41.1 mm

Commit message: sensor board work
Parts:
- removed DHT22: DHT22, adafruit:1X03
- removed JP1: JP1, adafruit:1X13
- removed JP2: JP2, adafruit:1X13
- removed MODE, RST: JST-XH-02-PIN-LONG-PAD, Rembrandt Electronics - JST XH Connectors v1-0:JST-XH-02-PACKAGE-LONG-PAD
- removed MOSFET1: 2N7000, 2N7000:TO92
- removed R1: 4.7K, resistor-power:HPS58
- removed R2: 2K, resistor-power:HPS58
- removed SENSOR: JST-XH-04-PIN-LONG-PAD, Rembrandt Electronics - JST XH Connectors v1-0:JST-XH-04-PACKAGE-LONG-PAD
- removed TEMP: JST-XH-03-PIN-LONG-PAD, Rembrandt Electronics - JST XH Connectors v1-0:JST-XH-03-PACKAGE-LONG-PAD
Connections:
- removed net 1WIRE: JP1.11, R1.2, TEMP.1
- removed net 3.3V: DHT22.1, JP2.11, R1.1, SENSOR.4, TEMP.3
- removed net DATA_T: DHT22.2, JP1.8
- removed net GND: JP1.12, MODE.2, MOSFET1.C, R2.1, RST.2
- removed net MODE: JP1.2, MODE.1
- removed net RST: JP1.3, RST.1
- removed net SCL: JP2.9, SENSOR.2
- removed net SDA: JP2.10, SENSOR.1
- removed net SENS_ENABLE: JP2.4, MOSFET1.B, R2.2
- removed net SENS_GND: DHT22.3, MOSFET1.E, SENSOR.3, TEMP.2
Routing:
- net SENS_GND: track 47.7 -> 0.00 mm
- net 3.3V: track 45.3 -> 0.00 mm
- net SCL: track 18.9 -> 0.00 mm
- net SENS_ENABLE: track 16.6 -> 0.00 mm
- net DATA_T: track 15.2 -> 0.00 mm
- net SDA: track 14.6 -> 0.00 mm
- net 1WIRE: track 14.5 -> 0.00 mm
- net RST: track 13.3 -> 0.00 mm
- net MODE: track 8.91 -> 0.00 mm
