File: TTGO_V11/hardware/KiCadSoil3/KiCadSoil3.sch (KiCad schematic (older format))
At the start: 11 parts, among them J1 Screw_Terminal_01x03, U1 ATtiny85-20PU, U2 TLC555CP

Commit message: include dallas
Parts:
- added U3: DS18B20, Package_TO_SOT_THT:TO-92_Inline, symbol Sensor_Temperature:DS18B20
Connections:
- wire segments 40 -> 41
Changed lines of the file:
@@
 	1    0    0    -1
 $EndComp
+$Comp
+L Sensor_Temperature:DS18B20 U3
+U 1 1 6089C6CE
+P 5450 1350
+F 0 "U3" V 5083 1350 50  0000 C CNN
+F 1 "DS18B20" V 5174 1350 50  0000 C CNN
+F 2 "Package_TO_SOT_THT:TO-92_Inline" H 4450 1100 50  0001 C CNN
+F 3 "http://datasheets.maximintegrated.com/en/ds/DS18B20.pdf" H 5300 1600 50  0001 C CNN
+	1    5450 1350
+	0    1    1    0
+$EndComp
+Wire Wire Line
+	5450 1650 4850 1650
+Connection ~ 4850 1650
+$Comp
+L power:GND #PWR0113
+U 1 1 6089E2E5
+P 5150 1350
+F 0 "#PWR0113" H 5150 1100 50  0001 C CNN
+F 1 "GND" H 5155 1177 50  0000 C CNN
+F 2 "" H 5150 1350 50  0001 C CNN
+F 3 "" H 5150 1350 50  0001 C CNN
+	1    5150 1350
+	0    1    1    0
+$EndComp
+$Comp
+L power:+3.3V #PWR0114
+U 1 1 6089EDA7
+P 5750 1350
+F 0 "#PWR0114" H 5750 1200 50  0001 C CNN
+F 1 "+3.3V" H 5765 1523 50  0000 C CNN
+F 2 "" H 5750 1350 50  0001 C CNN
+F 3 "" H 5750 1350 50  0001 C CNN
+	1    5750 1350
+	0    1    1    0
+$EndComp
 $EndSCHEMATC

Commit message: changes
Parts:
- U3: footprint Package_TO_SOT_THT:TO-92_Inline -> Package_TO_SOT_THT:TO-92_Inline_Wide
Changed lines of the file:
@@
 F 0 "U3" V 5083 1350 50  0000 C CNN
 F 1 "DS18B20" V 5174 1350 50  0000 C CNN
-F 2 "Package_TO_SOT_THT:TO-92_Inline" H 4450 1100 50  0001 C CNN
+F 2 "Package_TO_SOT_THT:TO-92_Inline_Wide" H 4450 1100 50  0001 C CNN
 F 3 "http://datasheets.maximintegrated.com/en/ds/DS18B20.pdf" H 5300 1600 50  0001 C CNN
 	1    5450 1350
