File: TTGO_V11/hardware/KiCadSoil3/KiCadSoil3.kicad_pcb (KiCad board)
At the start: 2 copper layers, 74.9 x 18.4 mm, 11 parts, among them J1 Screw_Terminal_01x03, U1 ATtiny85-20PU, U2 TLC555CP

Commit message: include dallas
Parts:
- added U3: DS18B20, Package_TO_SOT_THT:TO-92_Inline, F.Cu at (110.5, 33.7)
- U1: value ATtiny85-20PU -> ATtiny85
- moved C1 9.55 mm to (77.5, 48.3)
- moved C2 9.55 mm to (81.3, 38.7)
- moved J1 9.55 mm to (111.8, 43.8)
- moved R1 9.55 mm to (74.9, 45.1)
- moved R4 9.55 mm to (104.1, 48.3)
- moved U1 9.55 mm to (106.7, 37.5)
- moved U2 9.55 mm to (93.3, 37.5)
- moved C3 9.55 mm to (85.7, 48.3)
- moved D1 9.55 mm to (75.6, 36.2)
- moved R2 9.55 mm to (78.7, 41.3)
- moved R3 9.55 mm to (101.6, 48.3)
Routing:
- net /COUT: track 30.1 -> 40.1 mm
Other:
- board size 74.9 x 18.4 mm -> 83.8 x 19.7 mm

Commit message: add dallas
Parts:
- moved U3 1.91 mm to (112.4, 33.7)
Routing:
- net +3V3: track 43.1 -> 62.1 mm
- net /1-Wire: track 19.6 -> 27.8 mm
Other:
- outline, holes or cut-outs redrawn

Commit message: changes
Parts:
- U1: value ATtiny85 -> ATtiny85-20PU
- U3: footprint Package_TO_SOT_THT:TO-92_Inline -> Package_TO_SOT_THT:TO-92_Inline_Wide
- moved C1 0.90 mm to (76.8, 48.9)
- moved J1 0.90 mm to (111.1, 44.5)
- moved R4 0.90 mm to (103.5, 48.9)
- moved C2 0.90 mm to (80.6, 39.4)
- moved U1 0.90 mm to (106.0, 38.1)
- moved U2 0.90 mm to (92.7, 38.1)
- moved C3 0.90 mm to (85.1, 48.9)
- moved R3 0.90 mm to (101.0, 48.9)
- moved R2 0.90 mm to (78.1, 41.9)
- moved U3 0.64 mm to (113.0, 33.7)
- moved R1 0.63 mm to (74.9, 45.7)
- moved D1 0.63 mm to (74.9, 36.2)
Routing:
- net GND: track 0.64 -> 2.54 mm
- net /1-Wire: track 27.8 -> 29.3 mm
- net /AOUT: track 32.1 -> 30.7 mm
Other:
- board size 83.8 x 19.7 mm -> 84.5 x 19 mm
